File: eagle/WaterLevelController/waterLevelController.brd (EAGLE design)
At the start: 100 x 80 mm, 7 parts

Commit message: Routed
Parts:
- moved J2 11.5 mm to (49.5, 43.2), turned to 270 degrees
- moved J1 1.27 mm to (49.5, 19.1)
Connections:
- net N$7: now also U$3.JP1.3; no longer U$3.JP1.7
- net N$8: now also U$3.JP1.7; no longer U$3.JP2.3
- net N$9: now also U$3.JP1.6; no longer U$3.JP2.4
Routing:
- net N$2: track 0.00 -> 119.4 mm
- net N$4: track 0.00 -> 71.4 mm
- net N$9: track 0.00 -> 69.7 mm
- net N$7: track 0.00 -> 48.4 mm
- net N$8: track 0.00 -> 42.0 mm
- net N$1: track 0.00 -> 8.17 mm
- net N$6: track 0.00 -> 8.17 mm
- net N$5: track 0.00 -> 8.17 mm
- net N$3: track 0.00 -> 8.17 mm

Commit message: add pdf
Routing:
- net N$9: track 69.7 -> 71.5 mm
Changed lines of the file:
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@@
 <drawing>
 <settings>
-<setting alwaysvectorfont="no"/>
+<setting alwaysvectorfont="yes"/>
 <setting verticaltext="up"/>
 </settings>
@@
 <contactref element="J2" pad="1"/>
 <contactref element="J1" pad="1"/>
-<wire x1="26.59" y1="37.37" x2="26.59" y2="44.37" width="0.508" layer="1"/>
-<wire x1="27.94" y1="45.72" x2="26.59" y2="44.37" width="0.508" layer="1"/>
-<wire x1="27.94" y1="45.72" x2="49.53" y2="45.72" width="0.508" layer="1"/>
-<wire x1="26.59" y1="44.37" x2="10.24" y2="44.37" width="0.508" layer="1"/>
-<wire x1="10.24" y1="44.37" x2="10.16" y2="44.45" width="0.508" layer="1"/>
-<wire x1="10.16" y1="44.45" x2="9.525" y2="43.815" width="0.508" layer="1"/>
-<wire x1="9.525" y1="43.815" x2="9.525" y2="23.495" width="0.508" layer="1"/>
-<wire x1="9.525" y1="23.495" x2="10.16" y2="22.86" width="0.508" layer="1"/>
-<wire x1="10.16" y1="22.86" x2="33.02" y2="22.86" width="0.508" layer="1"/>
-<wire x1="33.02" y1="22.86" x2="33.02" y2="27.305" width="0.508" layer="1"/>
-<wire x1="33.02" y1="27.305" x2="32.385" y2="27.94" width="0.508" layer="1"/>
-<wire x1="49.53" y1="16.51" x2="34.29" y2="16.51" width="0.508" layer="1"/>
-<wire x1="34.29" y1="16.51" x2="33.02" y2="17.78" width="0.508" layer="1"/>
-<wire x1="33.02" y1="17.78" x2="33.02" y2="22.86" width="0.508" layer="1"/>
+<wire x1="26.59" y1="37.37" x2="26.59" y2="44.37" width="0.8128" layer="1"/>
+<wire x1="27.94" y1="45.72" x2="26.59" y2="44.37" width="0.8128" layer="1"/>
+<wire x1="27.94" y1="45.72" x2="49.53" y2="45.72" width="0.8128" layer="1"/>
+<wire x1="26.59" y1="44.37" x2="10.24" y2="44.37" width="0.8128" layer="1"/>
+<wire x1="10.24" y1="44.37" x2="10.16" y2="44.45" width="0.8128" layer="1"/>
+<wire x1="10.16" y1="44.45" x2="9.525" y2="43.815" width="0.8128" layer="1"/>
+<wire x1="9.525" y1="43.815" x2="9.525" y2="23.495" width="0.8128" layer="1"/>
+<wire x1="9.525" y1="23.495" x2="10.16" y2="22.86" width="0.8128" layer="1"/>
+<wire x1="10.16" y1="22.86" x2="33.02" y2="22.86" width="0.8128" layer="1"/>
+<wire x1="33.02" y1="22.86" x2="33.02" y2="27.305" width="0.8128" layer="1"/>
+<wire x1="33.02" y1="27.305" x2="32.385" y2="27.94" width="0.8128" layer="1"/>
+<wire x1="49.53" y1="16.51" x2="34.29" y2="16.51" width="0.8128" layer="1"/>
+<wire x1="34.29" y1="16.51" x2="33.02" y2="17.78" width="0.8128" layer="1"/>
+<wire x1="33.02" y1="17.78" x2="33.02" y2="22.86" width="0.8128" layer="1"/>
 </signal>
 <signal name="N$4">
@@
 <contactref element="J2" pad="2"/>
 <contactref element="J1" pad="2"/>
-<wire x1="29.845" y1="27.94" x2="29.845" y2="31.115" width="0.508" layer="1"/>
-<wire x1="36.1" y1="37.37" x2="41.99" y2="37.37" width="0.508" layer="1"/>
-<wire x1="29.845" y1="31.115" x2="36.1" y2="37.37" width="0.508" layer="1"/>
-<wire x1="41.99" y1="37.37" x2="41.99" y2="40.72" width="0.508" layer="1"/>
-<wire x1="41.99" y1="40.72" x2="44.45" y2="43.18" width="0.508" layer="1"/>
-<wire x1="44.45" y1="43.18" x2="49.53" y2="43.18" width="0.508" layer="1"/>
-<wire x1="41.99" y1="37.37" x2="41.99" y2="20.24" width="0.508" layer="1"/>
-<wire x1="41.99" y1="20.24" x2="43.18" y2="19.05" width="0.508" layer="1"/>
-<wire x1="43.18" y1="19.05" x2="49.53" y2="19.05" width="0.508" layer="1"/>
-<wire x1="29.845" y1="31.115" x2="27.94" y2="33.02" width="0.508" layer="1"/>
-<wire x1="27.94" y1="33.02" x2="19.05" y2="33.02" width="0.508" layer="1"/>
-<wire x1="19.05" y1="33.02" x2="17.86" y2="34.21" width="0.508" layer="1"/>
-<wire x1="17.86" y1="34.21" x2="17.86" y2="37.37" width="0.508" layer="1"/>
+<wire x1="29.845" y1="27.94" x2="29.845" y2="31.115" width="0.8128" layer="1"/>
+<wire x1="36.1" y1="37.37" x2="41.99" y2="37.37" width="0.8128" layer="1"/>
+<wire x1="29.845" y1="31.115" x2="36.1" y2="37.37" width="0.8128" layer="1"/>
+<wire x1="41.99" y1="37.37" x2="41.99" y2="40.72" width="0.8128" layer="1"/>
+<wire x1="41.99" y1="40.72" x2="44.45" y2="43.18" width="0.8128" layer="1"/>
+<wire x1="44.45" y1="43.18" x2="49.53" y2="43.18" width="0.8128" layer="1"/>
+<wire x1="41.99" y1="37.37" x2="41.99" y2="20.24" width="0.8128" layer="1"/>
+<wire x1="41.99" y1="20.24" x2="43.18" y2="19.05" width="0.8128" layer="1"/>
+<wire x1="43.18" y1="19.05" x2="49.53" y2="19.05" width="0.8128" layer="1"/>
+<wire x1="29.845" y1="31.115" x2="27.94" y2="33.02" width="0.8128" layer="1"/>
+<wire x1="27.94" y1="33.02" x2="19.05" y2="33.02" width="0.8128" layer="1"/>
+<wire x1="19.05" y1="33.02" x2="17.86" y2="34.21" width="0.8128" layer="1"/>
+<wire x1="17.86" y1="34.21" x2="17.86" y2="37.37" width="0.8128" layer="1"/>
 </signal>
 <signal name="N$7">
 <contactref element="HLK1" pad="P$4"/>
 <contactref element="U$3" pad="JP1.3"/>
-<wire x1="2.46" y1="37.37" x2="2.46" y2="8.97" width="0.508" layer="1"/>
-<wire x1="3.81" y1="7.62" x2="19.05" y2="7.62" width="0.508" layer="1"/>
-<wire x1="19.05" y1="7.62" x2="19.685" y2="6.985" width="0.508" layer="1"/>
-<wire x1="19.685" y1="6.985" x2="19.685" y2="5.08" width="0.508" layer="1"/>
-<wire x1="2.46" y1="8.97" x2="3.81" y2="7.62" width="0.508" layer="1"/>
+<wire x1="2.46" y1="37.37" x2="2.46" y2="8.97" width="0.8128" layer="1"/>
+<wire x1="3.81" y1="7.62" x2="19.05" y2="7.62" width="0.8128" layer="1"/>
+<wire x1="19.05" y1="7.62" x2="19.685" y2="6.985" width="0.8128" layer="1"/>
+<wire x1="19.685" y1="6.985" x2="19.685" y2="5.08" width="0.8128" layer="1"/>
+<wire x1="2.46" y1="8.97" x2="3.81" y2="7.62" width="0.8128" layer="1"/>
 </signal>
 <signal name="N$8">
 <contactref element="J1" pad="3"/>
 <contactref element="U$3" pad="JP1.7"/>
-<wire x1="49.53" y1="21.59" x2="53.34" y2="21.59" width="0.508" layer="1"/>
-<wire x1="53.34" y1="21.59" x2="53.34" y2="8.89" width="0.508" layer="1"/>
-<wire x1="53.34" y1="8.89" x2="52.07" y2="7.62" width="0.508" layer="1"/>
-<wire x1="52.07" y1="7.62" x2="31.75" y2="7.62" width="0.508" layer="1"/>
-<wire x1="31.75" y1="7.62" x2="29.845" y2="5.715" width="0.508" layer="1"/>
-<wire x1="29.845" y1="5.715" x2="29.845" y2="5.08" width="0.508" layer="1"/>
+<wire x1="49.53" y1="21.59" x2="53.34" y2="21.59" width="0.8128" layer="1"/>
+<wire x1="53.34" y1="21.59" x2="53.34" y2="8.89" width="0.8128" layer="1"/>
+<wire x1="53.34" y1="8.89" x2="52.07" y2="7.62" width="0.8128" layer="1"/>
+<wire x1="52.07" y1="7.62" x2="31.75" y2="7.62" width="0.8128" layer="1"/>
+<wire x1="31.75" y1="7.62" x2="29.845" y2="5.715" width="0.8128" layer="1"/>
+<wire x1="29.845" y1="5.715" x2="29.845" y2="5.08" width="0.8128" layer="1"/>
 </signal>
 <signal name="N$9">
 <contactref element="J2" pad="3"/>
 <contactref element="U$3" pad="JP1.6"/>
-<wire x1="49.53" y1="40.64" x2="54.61" y2="35.56" width="0.508" layer="1"/>
-<wire x1="54.61" y1="35.56" x2="54.61" y2="2.54" width="0.508" layer="1"/>
-<wire x1="54.61" y1="2.54" x2="27.94" y2="2.54" width="0.508" layer="1"/>
-<wire x1="27.94" y1="2.54" x2="27.305" y2="3.175" width="0.508" layer="1"/>
-<wire x1="27.305" y1="3.175" x2="27.305" y2="5.08" width="0.508" layer="1"/>
+<wire x1="49.53" y1="40.64" x2="55.88" y2="34.29" width="0.8128" layer="1"/>
+<wire x1="55.88" y1="34.29" x2="55.88" y2="2.54" width="0.8128" layer="1"/>
+<wire x1="55.88" y1="2.54" x2="27.94" y2="2.54" width="0.8128" layer="1"/>
+<wire x1="27.94" y1="2.54" x2="27.305" y2="3.175" width="0.8128" layer="1"/>
+<wire x1="27.305" y1="3.175" x2="27.305" y2="5.08" width="0.8128" layer="1"/>
 </signal>
 </signals>
